File: input.kicad_sch (KiCad schematic)
At the start: 3 parts, among them U8 PC817

Commit message: WIP
Parts:
- R8: footprint Resistor_SMD:R_1206_3216Metric -> Resistor_SMD:R_0603_1608Metric_Pad0.98x0.95mm_HandSolder; LCSC PN (none) -> C22978
- U8: footprint Package_DIP:DIP-4_W7.62mm -> Package_SO:SOP-4_4.4x2.6mm_P1.27mm; LCSC PN (none) -> C385060

Commit message: wip
Parts:
- renumbered R8 to R3, U8 to U3, input0 to input2
Changed lines of the file:
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@@
 		(on_board yes)
 		(dnp no)
-		(property "Reference" "U8"
+		(property "Reference" "U3"
 			(at 124.46 96.52 0)
 			(effects
@@
 		(dnp no)
 		(fields_autoplaced yes)
-		(property "Reference" "input0"
+		(property "Reference" "input2"
 			(at 152.4 88.9 0)
 			(effects
@@
 		(on_board yes)
 		(dnp no)
-		(property "Reference" "R8"
+		(property "Reference" "R3"
 			(at 135.89 82.55 90)
 			(effects

Commit message: wip
Parts:
- removed U3: PC817, Package_SO:SOP-4_4.4x2.6mm_P1.27mm, symbol Isolator:PC817
- added C18: 100n, Capacitor_SMD:C_0603_1608Metric_Pad1.08x0.95mm_HandSolder, symbol Device:C
- added U6: ELM453-TA-V, Package_SO:MFSOP6-5_4.4x3.6mm_P1.27mm, symbol Isolator:TLP137
Connections:
- net gnd: now also C18.2, U6.4
- net signal: now also U6.5
- net at R3.1: now also U6.1
- net at input2.1 (Pin_1): now also U6.3
- new net 3v3: C18.1, U6.6

Commit message: Fix missing clk line
Parts:
- renumbered C18 to C21, U6 to U17
Changed lines of the file:
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@@
 		(on_board yes)
 		(dnp no)
-		(property "Reference" "U6"
+		(property "Reference" "U17"
 			(at 124.46 78.74 0)
 			(effects
@@
 		(dnp no)
 		(fields_autoplaced yes)
-		(property "Reference" "C18"
+		(property "Reference" "C21"
 			(at 109.22 82.55 0)
 			(effects
